File: PCB/PEPSISat.kicad_pcb (KiCad board)
At the start: 2 copper layers, 3 parts, among them U1 STM32H747IITx, U2 RP2350A, U3 MT48LC16M16A2P

Commit message: Added RP2350 datasheet
Routing:
- net /FMC_D12: track 42.2 -> 44.9 mm
- net /FMC_D13: track 43.1 -> 40.6 mm
- net /FMC_D14: track 43.2 -> 41.0 mm
- net /FMC_D11: track 43.0 -> 45.2 mm
- net /FMC_D15: track 43.3 -> 41.4 mm
- net /FMC_D10: track 43.4 -> 45.3 mm
- net /FMC_D9: track 44.7 -> 45.9 mm
- net /FMC_A12: track 26.5 -> 27.7 mm
- net /FMC_D8: track 48.2 -> 48.9 mm

Commit message: KiCad
Parts:
- added J1: OV5640, Connector_PinHeader_2.54mm:PinHeader_2x09_P2.54mm_Horizontal, F.Cu at (73.3, 38.2)
- added U4: BMP280, Package_LGA:Bosch_LGA-8_2x2.5mm_P0.65mm_ClockwisePinNumbering, F.Cu at (69.0, 38.0)
- moved U2 61.6 mm to (62.4, 38.2), turned to 90 degrees
- moved U3 5.28 mm to (95.9, 59.2)
- moved U1 1.49 mm to (72.8, 59.7), turned to 90 degrees
Connections:
- U1 pad 114: unconnected-(U1-PG4-Pad114) -> /FMC.BA0
- U1 pad 115: unconnected-(U1-PG5-Pad115) -> /FMC.BA1
- U1 pad 118: unconnected-(U1-PG8-Pad118) -> /FMC.CLK
- U1 pad 122: unconnected-(U1-PC6-Pad122) -> /DCMI.D0
- U1 pad 123: unconnected-(U1-PC7-Pad123) -> /DCMI.D1
- U1 pad 124: unconnected-(U1-PC8-Pad124) -> /DCMI.D2
- U1 pad 125: unconnected-(U1-PC9-Pad125) -> /DCMI.D3
- U1 pad 127: unconnected-(U1-PA8-Pad127) -> /DCMI.XC
- U1 pad 128: unconnected-(U1-PA9-Pad128) -> /UART.TX
- U1 pad 129: unconnected-(U1-PA10-Pad129) -> /UART.RX
- U1 pad 130: unconnected-(U1-PA11-Pad130) -> /UART.CTS_{ST}-RTS_{RP}
- U1 pad 131: unconnected-(U1-PA12-Pad131) -> /UART.RTS_{ST}-CTS_{RP}
- U1 pad 146: unconnected-(U1-PD3-Pad146) -> /DCMI.D5
- U1 pad 161: unconnected-(U1-PG15-Pad161) -> /FMC.~{CAS}
- U1 pad 166: unconnected-(U1-PB7-Pad166) -> /DCMI.VS
- U1 pad 168: unconnected-(U1-PB8-Pad168) -> /DCMI.SCL
- U1 pad 169: unconnected-(U1-PB9-Pad169) -> /DCMI.SDA
- U1 pad 3: unconnected-(U1-PE4-Pad3) -> /DCMI.D4
- U1 pad 4: unconnected-(U1-PE5-Pad4) -> /DCMI.D6
- U1 pad 5: unconnected-(U1-PE6-Pad5) -> /DCMI.D7
- U1 pad 50: unconnected-(U1-PA5-Pad50) -> /DCMI.HS
- U1 pad 51: unconnected-(U1-PA6-Pad51) -> /DCMI.PC
- U1 pad 52: unconnected-(U1-PA7-Pad52) -> /FMC.~{WE}
- U1 pad 53: unconnected-(U1-PC4-Pad53) -> /FMC.~{CS}
- U1 pad 54: unconnected-(U1-PC5-Pad54) -> /FMC.CKE
- U1 pad 58: unconnected-(U1-PF11-Pad58) -> /FMC.~{RAS}
- U2 pad 14: unconnected-(U2-GPIO10-Pad14) -> Net-(U2-GPIO10)
- U2 pad 15: unconnected-(U2-GPIO11-Pad15) -> Net-(U2-GPIO11)
- U2 pad 16: unconnected-(U2-GPIO12-Pad16) -> Net-(U2-GPIO12)
- U2 pad 17: unconnected-(U2-GPIO13-Pad17) -> Net-(U2-GPIO13)
- U2 pad 2: unconnected-(U2-GPIO0-Pad2) -> /UART.TX
- U2 pad 3: unconnected-(U2-GPIO1-Pad3) -> /UART.RX
- U2 pad 4: unconnected-(U2-GPIO2-Pad4) -> /UART.RTS_{ST}-CTS_{RP}
- U2 pad 5: unconnected-(U2-GPIO3-Pad5) -> /UART.CTS_{ST}-RTS_{RP}
- U3 pad 15: unconnected-(U3-DQML-Pad15) -> /FMC.DQML
- U3 pad 16: unconnected-(U3-~{WE}-Pad16) -> /FMC.~{WE}
- U3 pad 17: unconnected-(U3-~{CAS}-Pad17) -> /FMC.~{CAS}
- U3 pad 18: unconnected-(U3-~{RAS}-Pad18) -> /FMC.~{RAS}
- U3 pad 19: unconnected-(U3-~{CS}-Pad19) -> /FMC.~{CS}
- U3 pad 20: unconnected-(U3-BA0-Pad20) -> /FMC.BA0
- U3 pad 21: unconnected-(U3-BA1-Pad21) -> /FMC.BA1
- U3 pad 37: unconnected-(U3-CKE-Pad37) -> /FMC.CKE
- U3 pad 38: unconnected-(U3-CLK-Pad38) -> /FMC.CLK
- U3 pad 39: unconnected-(U3-DQMH-Pad39) -> /FMC.DQMH
Routing:
- net /FMC_A4: track 78.7 -> 0.00 mm, vias 2 -> 1
- net /FMC_A5: track 73.1 -> 0.00 mm, vias 2 -> 1
- net /FMC_A10: track 50.9 -> 0.00 mm, vias 2 -> 1
- net /FMC_A6: track 49.6 -> 0.00 mm, vias 2 -> 1
- net /FMC_A7: track 49.1 -> 0.00 mm, vias 2 -> 1
- net /FMC_D8: track 48.9 -> 0.00 mm, vias 2 -> 1
- net /FMC_A8: track 48.6 -> 0.00 mm, vias 2 -> 1
- net /FMC_D4: track 48.3 -> 0.00 mm, vias 2 -> 1
- net /FMC_A9: track 48.1 -> 0.00 mm, vias 2 -> 1
- net /FMC_A3: track 48.0 -> 0.00 mm, vias 2 -> 1
- net /FMC_D6: track 47.8 -> 0.00 mm, vias 2 -> 1
- net /FMC_A11: track 46.9 -> 0.00 mm, vias 2 -> 1
- net /FMC_D9: track 45.9 -> 0.00 mm, vias 2 -> 1
- net /FMC_A2: track 45.9 -> 0.00 mm, vias 2 -> 1
- net /FMC_D10: track 45.3 -> 0.00 mm, vias 2 -> 1
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Other:
- board outline added: 60 x 100 mm

Commit message: KiCad
Parts:
- added R1: 4.7kR, Resistor_SMD:R_0603_1608Metric, B.Cu at (92.8, 42.3)
- added R2: 4.7kR, Resistor_SMD:R_0603_1608Metric, B.Cu at (92.8, 44.8)
- added U5: LSM6DSOXTR, LSM6DSOXTR:LGA-14L_STM, B.Cu at (98.0, 42.3)
- J1: value OV5640 -> Conn_02x09_Counter_Clockwise
Connections:
- U1 pad 95: unconnected-(U1-PD12-Pad95) -> GND
- U1 pad 96: unconnected-(U1-PD13-Pad96) -> Net-(U1-PD13)
